Commit message: B e cost function

File: Lite3/lite3_urdf/Lite3/urdf/Lite3.urdf (robot description, URDF)
Before this commit: robot MiniLiteV3, 18 links, 17 joints
Links:
- link TORSO: geometry collision box size=0.35 0.184 0.08

Commit message: tentativi camminata

File: Lite3/lite3_urdf/Lite3/urdf/Lite3.urdf (robot description, URDF)
Before this commit: robot MiniLiteV3, 18 links, 17 joints
Links:
- link TORSO: geometry collision box size=0.35 0.184 0.08; visual mesh filename=../meshes/Lite3.dae

Commit message: test

File: Lite3/lite3_urdf/Lite3/urdf/Lite3.urdf (robot description, URDF)
Before this commit: robot MiniLiteV3, 18 links, 17 joints
Links:
- link FL_FOOT: geometry collision sphere radius=0.01
- link FR_FOOT: geometry collision sphere radius=0.01
- link HL_FOOT: geometry collision sphere radius=0.01
- link HR_FOOT: geometry collision sphere radius=0.01

Commit message: fixes

File: Lite3/lite3_urdf/Lite3/urdf/Lite3.urdf (robot description, URDF)
Before this commit: robot MiniLiteV3, 18 links, 17 joints
Links:
- added link FL_FOOT2, mass 1E-12; collision sphere radius=0.01; visual sphere radius=0.01
- added link FR_FOOT2, mass 1E-12; collision sphere radius=0.01; visual sphere radius=0.01
- added link HL_FOOT2, mass 1E-12; collision sphere radius=0.01; visual sphere radius=0.01
- added link HR_FOOT2, mass 1E-12; collision sphere radius=0.01; visual sphere radius=0.01
- link HR_FOOT: geometry collision sphere radius=0.01; visual sphere radius=0.01
Joints:
- added joint FL_Ankle2: type fixed, parent FL_SHANK, child FL_FOOT2, origin xyz=-0.01 0 -0.225
- added joint FR_Ankle2: type fixed, parent FR_SHANK, child FR_FOOT2, origin xyz=-0.01 0 -0.225
- added joint HL_Ankle2: type fixed, parent HL_SHANK, child HL_FOOT2, origin xyz=-0.01 0 -0.225
- added joint HR_Ankle2: type fixed, parent HR_SHANK, child HR_FOOT2, origin xyz=-0.01 0 -0.225

File: Lite3/lite3_urdf/Lite3/urdf/ground.urdf (robot description, URDF)
Before this commit: robot ground_skeleton, 2 links, 1 joints
Links:
- link ground_link: mass 1.0 -> 0.00001
