Commit message: cammina

File: lite3_urdf/urdf/Lite3_backup.urdf (robot description, URDF)
Before this commit: robot MiniLiteV3, 18 links, 17 joints
Links:
- link HR_FOOT: geometry collision sphere radius=0.01

File: lite3_urdf/urdf/ground.urdf (robot description, URDF)
Before this commit: robot ground_skeleton, 2 links, 1 joints
Links:
- link ground_link: mass 0.00001 -> 100
