Commit message: updated collisions and removed some cache files

File: lite3_urdf/urdf/Lite3.urdf (robot description, URDF)
Before this commit: robot MiniLiteV3, 18 links, 17 joints
Links:
- link FL_FOOT: geometry visual sphere radius=0.01
- link FL_SHANK: geometry collision box size=0.02 0.02 0.28; visual box size=0.02 0.02 0.28
- link FR_FOOT: geometry 
- link FR_SHANK: geometry collision box size=0.02 0.02 0.28; visual box size=0.02 0.02 0.28
- link HL_FOOT: geometry 
- link HL_SHANK: geometry collision box size=0.02 0.02 0.28; visual box size=0.02 0.02 0.28
- link HR_FOOT: geometry visual sphere radius=0.01
- link HR_SHANK: geometry collision box size=0.02 0.02 0.28; visual box size=0.02 0.02 0.28

Commit message: prove nuova velocità

File: lite3_urdf/urdf/Lite3.urdf (robot description, URDF)
Before this commit: robot MiniLiteV3, 18 links, 17 joints
Links:
- link FL_FOOT: mass 1E-12 -> 1E-2
- link FR_FOOT: mass 1E-12 -> 1E-2
- link HL_FOOT: mass 1E-12 -> 1E-2
- link HR_FOOT: mass 1E-12 -> 1E-2

Commit message: Try camminata

File: lite3_urdf/urdf/Lite3.urdf (robot description, URDF)
Before this commit: robot MiniLiteV3, 18 links, 17 joints
Links:
- link FL_FOOT: mass 1E-12 -> 1E-2; geometry collision sphere radius=0.02
- link FR_FOOT: mass 1E-12 -> 1E-2; geometry collision sphere radius=0.02
- link HL_FOOT: mass 1E-12 -> 1E-2; geometry collision sphere radius=0.02
- link HR_FOOT: mass 1E-12 -> 1E-2; geometry collision sphere radius=0.02; visual sphere radius=0.02
Joints:
- joint FL_Ankle: origin xyz=0 0 -0.23 -> xyz=0 0 -0.21
- joint FR_Ankle: origin xyz=0 0 -0.23 -> xyz=0 0 -0.21
- joint HL_Ankle: origin xyz=0 0 -0.23 -> xyz=0 0 -0.21
- joint HR_Ankle: origin xyz=0 0 -0.23 -> xyz=0 0 -0.21

Commit message: tuning

File: lite3_urdf/urdf/Lite3.urdf (robot description, URDF)
Before this commit: robot MiniLiteV3, 18 links, 17 joints
Links:
- link FL_FOOT: geometry collision sphere radius=0.01; visual sphere radius=0.01

Commit message: clean-up

File: lite3_urdf/urdf/Lite3.urdf (robot description, URDF)
Before this commit: robot MiniLiteV3, 18 links, 17 joints
Links:
- link HR_FOOT: geometry collision sphere radius=0.02
